Commit message: Cambios al archivo .URDF

File: install/cibnor_sim/share/cibnor_sim/resource/cibnor_lidar_sensor.urdf (robot description, URDF)
Before this commit: robot robot, 11 links, 10 joints
Joints:
- joint base_link_to_hinge_BR: origin xyz=-0.21 -0.17 0 rpy=0 0.707108 -0.707105 -> xyz=-0.21 -0.17 0 rpy=1.5708006 0.0000019 -3.1415908
- joint base_link_to_hinge_FL: origin xyz=0.27 0.17 0 rpy=0 0.707108 -0.707105 -> xyz=0.27 0.17 0 rpy=1.5708006 0.0000019 -3.1415908
- joint base_link_to_hinge_FR: origin xyz=0.27 -0.17 0 rpy=0 -1.5708 0 -> xyz=0.27 -0.17 0 rpy=1.5708006 0.0000019 -3.1415908
- joint motor_BL: origin xyz=-0.21 0.25 0 rpy=1.57 0 0 -> xyz=0 0 -0.08 rpy=0 0 0
- joint motor_BR: origin xyz=-0.21 -0.25 0 rpy=1.57 0 0 -> xyz=0 0 -0.08 rpy=0 0 0
- joint motor_FL: origin xyz=0.27 0.25 0 rpy=1.57 0 0 -> xyz=0 0 0.08 rpy=0 0 0
- joint motor_FR: origin xyz=0.27 -0.25 0 rpy=1.57 0 0 -> xyz=0 0 -0.08 rpy=0 0 0

Commit message: Correcciones al archivo .URDF

File: install/cibnor_sim/share/cibnor_sim/resource/cibnor_lidar_sensor.urdf (robot description, URDF)
Before this commit: robot robot, 11 links, 10 joints
Links:
- added link ds_L; collision box size=0.01 0.02 0.01; visual box size=0.01 0.02 0.01
- added link ds_R; collision box size=0.01 0.02 0.01; visual box size=0.01 0.02 0.01
Joints:
- added joint base_link_to_ds_L: type fixed, parent base_link, child ds_L, origin xyz=0.326 0.05 -0.05 rpy=-0.1160253 0.2352153 0.4637244
- added joint base_link_to_ds_R: type fixed, parent base_link, child ds_R, origin xyz=0.326 -0.05 -0.05 rpy=0.1160253 0.2352153 -0.4637244
- joint base_link_to_hinge_BL: origin xyz=-0.21 0.17 0 rpy=-1.5708 0 3.1416 -> xyz=-0.21 0.17 0 rpy=1.5708006 0.0000019 -3.1415908
- joint motor_BL: origin xyz=0 0 -0.08 rpy=0 0 0 -> xyz=0 0 0.1 rpy=0 0 0
- joint motor_BR: origin xyz=0 0 -0.08 rpy=0 0 0 -> xyz=0 0 -0.1 rpy=0 0 0
- joint motor_FL: origin xyz=0 0 0.08 rpy=0 0 0 -> xyz=0 0 0.1 rpy=0 0 0
- joint motor_FR: origin xyz=0 0 -0.08 rpy=0 0 0 -> xyz=0 0 -0.1 rpy=0 0 0
- joint support_Lidar_to_lidar: origin xyz=0 0 0.2 rpy=0 0 0 -> xyz=0 0 0.09 rpy=0 0 0

Commit message: Modificacion de ruedas del archivo .wbt

File: install/cibnor_sim/share/cibnor_sim/resource/cibnor_lidar_sensor.urdf (robot description, URDF)
Before this commit: robot robot, 13 links, 12 joints
Links:
- link wheel_BL: geometry collision cylinder length=0.095 radius=0.175; visual cylinder length=0.095 radius=0.175
- link wheel_BR: geometry collision cylinder length=0.095 radius=0.175; visual cylinder length=0.095 radius=0.175
- link wheel_FL: geometry collision cylinder length=0.095 radius=0.175; visual cylinder length=0.095 radius=0.175
- link wheel_FR: geometry collision cylinder length=0.095 radius=0.175; visual cylinder length=0.095 radius=0.175
Joints:
- joint base_link_to_hinge_BL: origin xyz=-0.21 0.17 0 rpy=1.5708006 0.0000019 -3.1415908 -> xyz=-0.21 0.13 0 rpy=1.5708006 0.0000019 -3.1415908
- joint base_link_to_hinge_BR: origin xyz=-0.21 -0.17 0 rpy=1.5708006 0.0000019 -3.1415908 -> xyz=-0.21 -0.13 0 rpy=1.5708006 0.0000019 -3.1415908
- joint base_link_to_hinge_FL: origin xyz=0.27 0.17 0 rpy=1.5708006 0.0000019 -3.1415908 -> xyz=0.27 0.13 0 rpy=1.5708006 0.0000019 -3.1415908
- joint base_link_to_hinge_FR: origin xyz=0.27 -0.17 0 rpy=1.5708006 0.0000019 -3.1415908 -> xyz=0.27 -0.13 0 rpy=1.5708006 0.0000019 -3.1415908

Commit message: Implementacion de IMU y filtro de Kalman

File: install/cibnor_sim/share/cibnor_sim/resource/cibnor_lidar_sensor.urdf (robot description, URDF)
Before this commit: robot robot, 13 links, 12 joints
Links:
- added link imu; collision box size=0.022 0.017 0.005; visual box size=0.022 0.017 0.005
Joints:
- added joint base_link_to_imu: type fixed, parent base_link, child imu, origin xyz=0 0 0 rpy=0 0 0
